File: hardware/mcu/mcu.sch (KiCad schematic (older format))
At the start: 61 parts, among them J1 TYPE-C-31-M-12, J2 Conn_01x11, J3 Conn_01x11, J4 JST-PH Battery, J5 n_log, Q1 MUN5214DW1T1G, Q2 SI2301CDS-T1-GE3, Q3 SI2301CDS-T1-GE3, Q4 SI2301CDS-T1-GE3, SW1 Reset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

Commit message: Prototype scale v0.1
Parts:
- C7: value 1uF -> 10uF; LCSC Part Number C52923 -> C15525; Part Number CL05A105KA5NQNC -> CL05A106MQ5NUNC
- J1: LCSC Part Number (none) -> C165948; Part Number (none) -> TYPE-C-31-M-12
- R5: value 3k -> 3.3k; LCSC Part Number C25784 -> C25890; Part Number 0402WGF3001TCE -> 0402WGF3301TCE
- SW1: value Reset -> SKRKAEE020
- SW2: LCSC Part Number (none) -> C92660; Part Number (none) -> K3-1235S-F1
- SW3: value Boot -> SKRKAEE020
- U1: LCSC Part Number (none) -> C193707; Part Number (none) -> ESP32-PICO-D4
- U3: LCSC Part Number (none) -> C558442; Part Number (none) -> TPUSBLC6-2SC6
- U4: footprint Package_TO_SOT_SMD:SOT-23-5_HandSoldering -> Package_TO_SOT_SMD:SOT-23-5; LCSC C32574 -> (none); LCSC Part Number (none) -> C32574; Part Number (none) -> TP4054
Connections:
- net batt_adc: now also U1.8 (SENSOR_VN); no longer U1.13 (IO33)
- net io12: now also J2.9 (Pin_9); no longer J2.10 (Pin_10)
- net io13: now also J2.10 (Pin_10); no longer J2.11 (Pin_11)
- net io14: now also J2.11 (Pin_11); no longer J2.9 (Pin_9)
- net io18: now also J3.5 (Pin_5); no longer J3.4 (Pin_4)
- net io19: now also J3.7 (Pin_7); no longer J3.6 (Pin_6)
- net io21: now also J3.9 (Pin_9); no longer J3.7 (Pin_7)
- net io23: now also J3.4 (Pin_4); no longer J3.9 (Pin_9)
- net io25: now also J2.4 (Pin_4); no longer J2.6 (Pin_6)
- net io26: now also J2.5 (Pin_5); no longer J2.7 (Pin_7)
- net io32: now also J2.2 (Pin_2); no longer J2.5 (Pin_5)
- net io34: now also J2.6 (Pin_6); no longer J2.3 (Pin_3)
- net io35: now also J2.1 (Pin_1); no longer J2.4 (Pin_4)
- net io5: now also J3.6 (Pin_6); no longer J3.5 (Pin_5)
- net sensor_capn: now also J2.7 (Pin_7); no longer J2.1 (Pin_1)
- net sensor_capp: now also C20.2, R12.1, R13.2
- net sensor_vp: no longer C20.2, R12.1, R13.2
- removed net sensor_vn: J2.2 (Pin_2), U1.8 (SENSOR_VN)
- new net io33: J2.3 (Pin_3), U1.13 (IO33)
- no-connect marks 23 -> 24
Other:
- note added: "This defaults the DC-\nDC to use powersave\nmode which is likely\nnot sufficient for \nWiFi. Jumper to \nallow cutting in case \nit can't even boot"
- note added: "USB-UART"
- note removed: "5V boost for peripherals"
- note removed: "Check serial chip vdd. Should it just hook up to 3.3v instead of vbus?"
- note removed: "Extra indicator LEDs?"
- note removed: "Fuse on battery?"
- note removed: "LDO for peripherals"
- note removed: "Pin 1 markers for JLC"
- note removed: "Voltage dividers for battery and USB sense"
- moved on the sheet: AE1, C10, C18, C5, J2, J3, J4, J5, JP1, R14, TP1, U1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

Commit message: Working scale + controller
Parts:
- removed C17: 100nF, Capacitor_SMD:C_0402_1005Metric, symbol Device:C_Small
Connections:
- net en_switched_3v3: no longer U1.25 (IO16)
- new net io16: U1.25 (IO16)
Other:
- note added: "Add battery discharge protection"
- note added: "Brownout on LDO? Even more caps?"
- note added: "CAN'T USE io16 IT IS FLASH"
- note added: "CAN'T USE io17 IT IS FLASH"
- note added: "LDO is only 200MA so it browns out sometimes"
- note added: "VPP(16) NEEDS CAP TO PROGRAM EEPROM"
Changed lines of the file:
@@
 Text Label 10250 3800 0    50   ~ 0
 io0
-$Comp
-L Device:C_Small C17
-U 1 1 6118867F
-P 10050 3850
-F 0 "C17" V 10100 3700 50  0000 L CNN
-F 1 "100nF" V 10100 3900 50  0000 L CNN
-F 2 "Capacitor_SMD:C_0402_1005Metric" H 10050 3850 50  0001 C CNN
-F 3 "~" H 10050 3850 50  0001 C CNN
-F 4 "CL05B104KO5NNNC" H 10050 3850 50  0001 C CNN "Part Number"
-F 5 "C1525" H 10050 3850 50  0001 C CNN "LCSC Part Number"
-	1    10050 3850
-	0    1    1    0
-$EndComp
-Wire Wire Line
-	10150 3850 10250 3850
-Wire Wire Line
-	10250 3850 10250 3700
-Wire Wire Line
-	9950 3850 9850 3850
-Wire Wire Line
-	9850 3850 9850 3800
 Text Label 10600 2550 0    50   ~ 0
 io0
@@
 Wire Wire Line
 	9750 3800 9850 3800
-Connection ~ 9850 3800
 Wire Wire Line
 	9850 3800 9850 3700
@@
 Wire Wire Line
 	10300 1900 10300 2000
-Text Label 4100 6250 0    50   ~ 0
+Text Label 4150 6250 0    50   ~ 0
 io16
 Text Label 9150 3450 2    50   ~ 0
@@
 	4100 7150 3900 7150
 NoConn ~ 3900 7150
+Text Notes 12450 1050 0    79   ~ 0
+CAN'T USE io16 IT IS FLASH
+Text Notes 12600 1400 0    79   ~ 0
+CAN'T USE io17 IT IS FLASH
+Text Notes 12350 1700 0    79   ~ 0
+VPP(16) NEEDS CAP TO PROGRAM EEPROM
+Text Notes 12450 500  0    79   ~ 0
+Brownout on LDO? Even more caps?
+Text Notes 13250 600  0    79   ~ 0
+LDO is only 200MA so it browns out sometimes
+Wire Wire Line
+	10250 3700 10250 3800
+Text Notes 12350 2050 0    79   ~ 0
+Add battery discharge protection
 $EndSCHEMATC
